File: teensy_3-6sch.sch (EAGLE design)
At the start: 0 parts

Commit message: Routed everything
Parts:
- added R1, R3, R5, R7: 6.8k, rcl:R-EU_M0805
- added R2, R4, R6, R8: 200, rcl:R-EU_M0805
- added SV1, SV10, SV11, SV12, SV13, SV2, SV3, SV4, SV5, SV6, SV7, SV8, SV9: (no value), con-lstb:MA04-1
- added U$1, U$2: TEENSY_36, misc_luke:TEENSY_36
- added U$10, U$11, U$28, U$29, U$30, U$31, U$32, U$33, U$34, U$35, U$4, U$5, U$6, U$7, U$8, U$9: S3BPH, misc_luke:S3BPH
- added U$12, U$13, U$14, U$15, U$16, U$17, U$18, U$19, U$20, U$21, U$22, U$23, U$24, U$25, U$26, U$27: CPC1706, misc_luke:CPC1706
- added U$3: MAX232_BREAKOUT, misc_luke:MAX232_BREAKOUT
Connections:
- new net +3V3: SV3.3, SV3.4, U$10.1, U$11.1, U$29.1, U$30.1, U$31.1, U$4.1, U$5.1, U$6.1, U$7.1, U$8.1, U$9.1
- new net +5V: SV1.4, SV12.4, SV2.3, SV2.4, U$1G$1.VIN, U$28.1, U$2G$1.VIN, U$3.VCC, U$32.1, U$33.1, U$34.1, U$35.1
- new net ACT1: U$12.IN+, U$1G$3.D24
- new net ACT10: U$1G$2.D2, U$21.IN+
- new net ACT11: U$1G$2.D3, U$22.IN+
- new net ACT12: U$1G$2.D4, U$23.IN+
- new net ACT13: U$1G$2.D5, U$24.IN+
- new net ACT14: U$1G$2.D6, U$25.IN+
- new net ACT15: U$1G$2.D14/A0, U$26.IN+
- new net ACT16: U$1G$2.D15/A1, U$27.IN+
- new net ACT2: U$13.IN+, U$1G$3.D25
- new net ACT3: U$14.IN+, U$1G$3.D26
- new net ACT4: U$15.IN+, U$1G$3.D27
- new net ACT5: U$16.IN+, U$1G$3.D28
- new net ACT6: U$17.IN+, U$1G$3.D29
- new net ACT7: U$18.IN+, U$1G$3.D30
- new net ACT8: U$19.IN+, U$1G$3.D31/A12
- new net ACT9: U$1G$3.D32/A13, U$20.IN+
- new net ADC_CURRENT: U$1G$3.DAC1, U$29.3
- new net ADC_DISTANCE: U$1G$2.D19/A5, U$32.3
- new net ADC_PRESSURE: U$1G$2.D22/A8, U$31.3
- new net ADC_TEMP: U$1G$2.D21/A7, U$30.3
- new net AO1: SV4.1, U$12.OUT2
- new net AO10: SV8.3, U$21.OUT2
- new net AO11: SV9.1, U$22.OUT2
- new net AO12: SV9.3, U$23.OUT2
- new net AO13: SV10.1, U$24.OUT2
- new net AO14: SV10.3, U$25.OUT2
- new net AO15: SV11.1, U$26.OUT2
- new net AO16: SV11.3, U$27.OUT2
- new net AO2: SV4.3, U$13.OUT2
- new net AO3: SV5.1, U$14.OUT2
- new net AO4: SV5.3, U$15.OUT2
- new net AO5: SV6.1, U$16.OUT2
- new net AO6: SV6.3, U$17.OUT2
- new net AO7: SV7.1, U$18.OUT2
- new net AO8: SV7.3, U$19.OUT2
- new net AO9: SV8.1, U$20.OUT2
- new net ENC1: R1.2, U$1G$2.D17/A3, U$28.3
- new net ENC2: R3.2, U$1G$2.D18/A4, U$33.3
- new net ENC3: R5.2, U$1G$2.D7, U$34.3
- new net ENC4: R7.2, U$1G$2.D8, U$35.3
- new net GND: R1.1, R2.1, R3.1, R4.1, R5.1, R6.1, R7.1, R8.1, SV1.1, SV12.1, SV2.1, SV2.2, SV3.1, SV3.2, U$10.2, U$11.2, U$12.IN-, U$13.IN-, U$14.IN-, U$15.IN-, U$16.IN-, U$17.IN-, U$18.IN-, U$19.IN-, U$1G$1.AGND, U$1G$1.GND, U$1G$1.GND1, U$20.IN-, U$21.IN-, U$22.IN-, U$23.IN-, U$24.IN-, U$25.IN-, U$26.IN-, U$27.IN-, U$29.2, U$2G$1.AGND, U$2G$1.GND, U$2G$1.GND1, U$3.GND, U$30.2, U$31.2, U$32.2, U$4.2, U$5.2, U$6.2, U$7.2, U$8.2, U$9.2
- new net IMU1RX: SV12.2, U$3.T1OUT
- new net IMU1TX: SV12.3, U$3.R1IN
- new net IMU2RX: SV1.2, U$3.T2OUT
- new net IMU2TX: SV1.3, U$3.R2IN
- new net N$1: R2.2, U$28.2
- new net N$14: U$1G$2.D9
- new net N$15: U$1G$2.D10
- new net N$16: U$1G$2.D11
- new net N$17: U$1G$2.D12
- new net N$18: U$1G$2.D13
- new net N$2: R4.2, U$33.2
- new net N$21: U$1G$2.D16/A2
- new net N$25: U$1G$2.D20/A6
- new net N$28: U$1G$2.D23/A9
- new net N$3: R6.2, U$34.2
- new net N$4: R8.2, U$35.2
- new net POT1: U$1G$3.D33/A14, U$8.3
- new net POT2: U$1G$3.D34/A15, U$4.3
- new net POT3: U$1G$3.D35/A16, U$5.3
- new net POT4: U$1G$3.D36/A17, U$6.3
- new net POT5: U$1G$3.D37/A18, U$7.3
- new net POT6: U$1G$3.D38/A19, U$9.3
- new net POT7: U$10.3, U$1G$3.D39/A20
- new net POT8: U$11.3, U$1G$3.DAC0
- new net RX1: U$1G$2.D0, U$2G$2.D1
- new net RX2: U$2G$2.D7, U$3.R1OUT
- new net RX3: U$2G$2.D5, U$3.R2OUT
- new net TX1: U$1G$2.D1, U$2G$2.D0
- new net TX2: U$2G$2.D8, U$3.T1IN
- new net TX3: U$2G$2.D6, U$3.T2IN
- new net V+: SV13.3, SV13.4, U$12.OUT1, U$13.OUT1, U$14.OUT1, U$15.OUT1, U$16.OUT1, U$17.OUT1, U$18.OUT1, U$19.OUT1, U$20.OUT1, U$21.OUT1, U$22.OUT1, U$23.OUT1, U$24.OUT1, U$25.OUT1, U$26.OUT1, U$27.OUT1
- new net V-: SV10.2, SV10.4, SV11.2, SV11.4, SV13.1, SV13.2, SV4.2, SV4.4, SV5.2, SV5.4, SV6.2, SV6.4, SV7.2, SV7.4, SV8.2, SV8.4, SV9.2, SV9.4
Other:
- note added: "Current"
- note added: "Distance"
- note added: "Pressure"
- note added: "Teensy Master"
- note added: "Teensy Slave"
- note added: "Temp"
